Commit message: end urdf model

File: arm_description/urdf/arm.urdf.xacro (robot description, xacro)
@@ -178,5 +178,5 @@
     <!-- ________________________________________________________________________________ -->
     <link name="hand_link">
-        <xacro:default_inertial mass="0.2"/>
+        <xacro:default_inertial mass="0.1"/>
         <visual>
             <origin xyz="0.0 0.0 0.0" rpy="0.0 0.0 0.0"/>
@@ -192,4 +192,384 @@
             <geometry>
                 <mesh filename="package://arm_description/mesh/hand.STL" scale="0.3 0.3 0.3"/>
+            </geometry>
+        </collision>
+    </link>
+    <!-- ________________________________________________________________________________ -->
+    <link name="thumb_link">
+        <xacro:default_inertial mass="0.01"/>
+        <visual>
+            <origin xyz="0.0 0.0 0.0" rpy="0.0 0.0 0.0"/>
+            <geometry>
+                <mesh filename="package://arm_description/mesh/joint_thumb.STL" scale="0.3 0.3 0.3"/>
+            </geometry>
+            <material name="LightGrey">
+                <color rgba="0.7 0.7 0.7 1.0"/>
+            </material>
+        </visual>
+        <collision>
+            <origin xyz="0.0 0.0 0.0" rpy="0.0 0.0 0.0"/>
+            <geometry>
+                <mesh filename="package://arm_description/mesh/joint_thumb.STL" scale="0.3 0.3 0.3"/>
+            </geometry>
+        </collision>
+    </link>
+    <!-- ________________________________________________________________________________ -->
+    <link name="thumb_finger_link">
+        <xacro:default_inertial mass="0.01"/>
+        <visual>
+            <origin xyz="0.0 0.0 0.0" rpy="0.0 0.0 0.0"/>
+            <geometry>
+                <mesh filename="package://arm_description/mesh/joint_finger.STL" scale="0.3 0.3 0.3"/>
+            </geometry>
+            <material name="LightGrey">
+                <color rgba="0.7 0.7 0.7 1.0"/>
+            </material>
+        </visual>
+        <collision>
+            <origin xyz="0.0 0.0 0.0" rpy="0.0 0.0 0.0"/>
+            <geometry>
+                <mesh filename="package://arm_description/mesh/joint_finger_thumb.STL" scale="0.3 0.3 0.3"/>
+            </geometry>
+        </collision>
+    </link>
+    <!-- ________________________________________________________________________________ -->
+    <link name="phalanx_thumb_1_link">
+        <xacro:default_inertial mass="0.01"/>
+        <visual>
+            <origin xyz="0.0 0.0 0.0" rpy="0.0 0.0 0.0"/>
+            <geometry>
+                <mesh filename="package://arm_description/mesh/phalanx_thumb_1.STL" scale="0.3 0.3 0.3"/>
+            </geometry>
+            <material name="LightGrey">
+                <color rgba="0.7 0.7 0.7 1.0"/>
+            </material>
+        </visual>
+        <collision>
+            <origin xyz="0.0 0.0 0.0" rpy="0.0 0.0 0.0"/>
+            <geometry>
+                <mesh filename="package://arm_description/mesh/phalanx_thumb_1.STL" scale="0.3 0.3 0.3"/>
+            </geometry>
+        </collision>
+    </link>
+    <!-- ________________________________________________________________________________ -->
+    <link name="phalanx_thumb_2_link">
+        <xacro:default_inertial mass="0.01"/>
+        <visual>
+            <origin xyz="0.0 0.0 0.0" rpy="0.0 0.0 0.0"/>
+            <geometry>
+                <mesh filename="package://arm_description/mesh/phalanx_thumb_2.STL" scale="0.3 0.3 0.3"/>
+            </geometry>
+            <material name="LightGrey">
+                <color rgba="0.7 0.7 0.7 1.0"/>
+            </material>
+        </visual>
+        <collision>
+            <origin xyz="0.0 0.0 0.0" rpy="0.0 0.0 0.0"/>
+            <geometry>
+                <mesh filename="package://arm_description/mesh/phalanx_thumb_2.STL" scale="0.3 0.3 0.3"/>
+            </geometry>
+        </collision>
+    </link>
+    <!-- ________________________________________________________________________________ -->
+    <link name="lit_finger_link">
+        <xacro:default_inertial mass="0.01"/>
+        <visual>
+            <origin xyz="0.0 0.0 0.0" rpy="0.0 0.0 0.0"/>
+            <geometry>
+                <mesh filename="package://arm_description/mesh/joint_finger.STL" scale="0.3 0.3 0.3"/>
+            </geometry>
+            <material name="LightGrey">
+                <color rgba="0.7 0.7 0.7 1.0"/>
+            </material>
+        </visual>
+        <collision>
+            <origin xyz="0.0 0.0 0.0" rpy="0.0 0.0 0.0"/>
+            <geometry>
+                <mesh filename="package://arm_description/mesh/joint_finger.STL" scale="0.3 0.3 0.3"/>
+            </geometry>
+        </collision>
+    </link>
+    <!-- ________________________________________________________________________________ -->
+    <link name="phalanx_lit_finger_1_link">
+        <xacro:default_inertial mass="0.01"/>
+        <visual>
+            <origin xyz="0.0 0.0 0.0" rpy="0.0 0.0 0.0"/>
+            <geometry>
+                <mesh filename="package://arm_description/mesh/phalanx_lit_finger_1.STL" scale="0.3 0.3 0.3"/>
+            </geometry>
+            <material name="LightGrey">
+                <color rgba="0.7 0.7 0.7 1.0"/>
+            </material>
+        </visual>
+        <collision>
+            <origin xyz="0.0 0.0 0.0" rpy="0.0 0.0 0.0"/>
+            <geometry>
+                <mesh filename="package://arm_description/mesh/phalanx_lit_finger_1.STL" scale="0.3 0.3 0.3"/>
+            </geometry>
+        </collision>
+    </link>
+    <!-- ________________________________________________________________________________ -->
+    <link name="phalanx_lit_finger_2_link">
+        <xacro:default_inertial mass="0.01"/>
+        <visual>
+            <origin xyz="0.0 0.0 0.0" rpy="0.0 0.0 0.0"/>
+            <geometry>
+                <mesh filename="package://arm_description/mesh/phalanx_lit_finger_2.STL" scale="0.3 0.3 0.3"/>
+            </geometry>
+            <material name="LightGrey">
+                <color rgba="0.7 0.7 0.7 1.0"/>
+            </material>
+        </visual>
+        <collision>
+            <origin xyz="0.0 0.0 0.0" rpy="0.0 0.0 0.0"/>
+            <geometry>
+                <mesh filename="package://arm_description/mesh/phalanx_lit_finger_2.STL" scale="0.3 0.3 0.3"/>
+            </geometry>
+        </collision>
+    </link>
+    <!-- ________________________________________________________________________________ -->
+    <link name="phalanx_lit_finger_3_link">
+        <xacro:default_inertial mass="0.01"/>
+        <visual>
+            <origin xyz="0.0 0.0 0.0" rpy="0.0 0.0 0.0"/>
+            <geometry>
+                <mesh filename="package://arm_description/mesh/phalanx_lit_finger_3.STL" scale="0.3 0.3 0.3"/>
+            </geometry>
+            <material name="LightGrey">
+                <color rgba="0.7 0.7 0.7 1.0"/>
+            </material>
+        </visual>
+        <collision>
+            <origin xyz="0.0 0.0 0.0" rpy="0.0 0.0 0.0"/>
+            <geometry>
+                <mesh filename="package://arm_description/mesh/phalanx_lit_finger_3.STL" scale="0.3 0.3 0.3"/>
+            </geometry>
+        </collision>
+    </link>
+    <!-- ________________________________________________________________________________ -->
+    <link name="ring_finger_link">
+        <xacro:default_inertial mass="0.01"/>
+        <visual>
+            <origin xyz="0.0 0.0 0.0" rpy="0.0 0.0 0.0"/>
+            <geometry>
+                <mesh filename="package://arm_description/mesh/joint_finger.STL" scale="0.3 0.3 0.3"/>
+            </geometry>
+            <material name="LightGrey">
+                <color rgba="0.7 0.7 0.7 1.0"/>
+            </material>
+        </visual>
+        <collision>
+            <origin xyz="0.0 0.0 0.0" rpy="0.0 0.0 0.0"/>
+            <geometry>
+                <mesh filename="package://arm_description/mesh/joint_finger.STL" scale="0.3 0.3 0.3"/>
+            </geometry>
+        </collision>
+    </link>
+    <!-- ________________________________________________________________________________ -->
+    <link name="phalanx_ring_finger_1_link">
+        <xacro:default_inertial mass="0.01"/>
+        <visual>
+            <origin xyz="0.0 0.0 0.0" rpy="0.0 0.0 0.0"/>
+            <geometry>
+                <mesh filename="package://arm_description/mesh/phalanx_finger_1.STL" scale="0.3 0.3 0.3"/>
+            </geometry>
+            <material name="LightGrey">
+                <color rgba="0.7 0.7 0.7 1.0"/>
+            </material>
+        </visual>
+        <collision>
+            <origin xyz="0.0 0.0 0.0" rpy="0.0 0.0 0.0"/>
+            <geometry>
+                <mesh filename="package://arm_description/mesh/phalanx_finger_1.STL" scale="0.3 0.3 0.3"/>
+            </geometry>
+        </collision>
+    </link>
+    <!-- ________________________________________________________________________________ -->
+    <link name="phalanx_ring_finger_2_link">
+        <xacro:default_inertial mass="0.01"/>
+        <visual>
+            <origin xyz="0.0 0.0 0.0" rpy="0.0 0.0 0.0"/>
+            <geometry>
+                <mesh filename="package://arm_description/mesh/phalanx_finger_2.STL" scale="0.3 0.3 0.3"/>
+            </geometry>
+            <material name="LightGrey">
+                <color rgba="0.7 0.7 0.7 1.0"/>
+            </material>
+        </visual>
+        <collision>
+            <origin xyz="0.0 0.0 0.0" rpy="0.0 0.0 0.0"/>
+            <geometry>
+                <mesh filename="package://arm_description/mesh/phalanx_finger_2.STL" scale="0.3 0.3 0.3"/>
+            </geometry>
+        </collision>
+    </link>
+    <!-- ________________________________________________________________________________ -->
+    <link name="phalanx_ring_finger_3_link">
+        <xacro:default_inertial mass="0.01"/>
+        <visual>
+            <origin xyz="0.0 0.0 0.0" rpy="0.0 0.0 0.0"/>
+            <geometry>
+                <mesh filename="package://arm_description/mesh/phalanx_finger_3.STL" scale="0.3 0.3 0.3"/>
+            </geometry>
+            <material name="LightGrey">
+                <color rgba="0.7 0.7 0.7 1.0"/>
+            </material>
+        </visual>
+        <collision>
+            <origin xyz="0.0 0.0 0.0" rpy="0.0 0.0 0.0"/>
+            <geometry>
+                <mesh filename="package://arm_description/mesh/phalanx_finger_3.STL" scale="0.3 0.3 0.3"/>
+            </geometry>
+        </collision>
+    </link>
+    <!-- ________________________________________________________________________________ -->
+    <link name="mid_finger_link">
+        <xacro:default_inertial mass="0.01"/>
+        <visual>
+            <origin xyz="0.0 0.0 0.0" rpy="0.0 0.0 0.0"/>
+            <geometry>
+                <mesh filename="package://arm_description/mesh/joint_finger.STL" scale="0.3 0.3 0.3"/>
+            </geometry>
+            <material name="LightGrey">
+                <color rgba="0.7 0.7 0.7 1.0"/>
+            </material>
+        </visual>
+        <collision>
+            <origin xyz="0.0 0.0 0.0" rpy="0.0 0.0 0.0"/>
+            <geometry>
+                <mesh filename="package://arm_description/mesh/joint_finger.STL" scale="0.3 0.3 0.3"/>
+            </geometry>
+        </collision>
+    </link>
+    <!-- ________________________________________________________________________________ -->
+    <link name="phalanx_mid_finger_1_link">
+        <xacro:default_inertial mass="0.01"/>
+        <visual>
+            <origin xyz="0.0 0.0 0.0" rpy="0.0 0.0 0.0"/>
+            <geometry>
+                <mesh filename="package://arm_description/mesh/phalanx_finger_1.STL" scale="0.3 0.3 0.3"/>
+            </geometry>
+            <material name="LightGrey">
+                <color rgba="0.7 0.7 0.7 1.0"/>
+            </material>
+        </visual>
+        <collision>
+            <origin xyz="0.0 0.0 0.0" rpy="0.0 0.0 0.0"/>
+            <geometry>
+                <mesh filename="package://arm_description/mesh/phalanx_finger_1.STL" scale="0.3 0.3 0.3"/>
+            </geometry>
+        </collision>
+    </link>
+    <!-- ________________________________________________________________________________ -->
+    <link name="phalanx_mid_finger_2_link">
+        <xacro:default_inertial mass="0.01"/>
+        <visual>
+            <origin xyz="0.0 0.0 0.0" rpy="0.0 0.0 0.0"/>
+            <geometry>
+                <mesh filename="package://arm_description/mesh/phalanx_finger_2.STL" scale="0.3 0.3 0.3"/>
+            </geometry>
+            <material name="LightGrey">
+                <color rgba="0.7 0.7 0.7 1.0"/>
+            </material>
+        </visual>
+        <collision>
+            <origin xyz="0.0 0.0 0.0" rpy="0.0 0.0 0.0"/>
+            <geometry>
+                <mesh filename="package://arm_description/mesh/phalanx_finger_2.STL" scale="0.3 0.3 0.3"/>
+            </geometry>
+        </collision>
+    </link>
+    <!-- ________________________________________________________________________________ -->
+    <link name="phalanx_mid_finger_3_link">
+        <xacro:default_inertial mass="0.01"/>
+        <visual>
+            <origin xyz="0.0 0.0 0.0" rpy="0.0 0.0 0.0"/>
+            <geometry>
+                <mesh filename="package://arm_description/mesh/phalanx_finger_3.STL" scale="0.3 0.3 0.3"/>
+            </geometry>
+            <material name="LightGrey">
+                <color rgba="0.7 0.7 0.7 1.0"/>
+            </material>
+        </visual>
+        <collision>
+            <origin xyz="0.0 0.0 0.0" rpy="0.0 0.0 0.0"/>
+            <geometry>
+                <mesh filename="package://arm_description/mesh/phalanx_finger_3.STL" scale="0.3 0.3 0.3"/>
+            </geometry>
+        </collision>
+    </link>
+    <!-- ________________________________________________________________________________ -->
+    <link name="forefinger_link">
+        <xacro:default_inertial mass="0.01"/>
+        <visual>
+            <origin xyz="0.0 0.0 0.0" rpy="0.0 0.0 0.0"/>
+            <geometry>
+                <mesh filename="package://arm_description/mesh/joint_finger.STL" scale="0.3 0.3 0.3"/>
+            </geometry>
+            <material name="LightGrey">
+                <color rgba="0.7 0.7 0.7 1.0"/>
+            </material>
+        </visual>
+        <collision>
+            <origin xyz="0.0 0.0 0.0" rpy="0.0 0.0 0.0"/>
+            <geometry>
+                <mesh filename="package://arm_description/mesh/joint_finger.STL" scale="0.3 0.3 0.3"/>
+            </geometry>
+        </collision>
+    </link>
+    <!-- ________________________________________________________________________________ -->
+    <link name="phalanx_forefinger_1_link">
+        <xacro:default_inertial mass="0.01"/>
+        <visual>
+            <origin xyz="0.0 0.0 0.0" rpy="0.0 0.0 0.0"/>
+            <geometry>
+                <mesh filename="package://arm_description/mesh/phalanx_finger_1.STL" scale="0.3 0.3 0.3"/>
+            </geometry>
+            <material name="LightGrey">
+                <color rgba="0.7 0.7 0.7 1.0"/>
+            </material>
+        </visual>
+        <collision>
+            <origin xyz="0.0 0.0 0.0" rpy="0.0 0.0 0.0"/>
+            <geometry>
+                <mesh filename="package://arm_description/mesh/phalanx_finger_1.STL" scale="0.3 0.3 0.3"/>
+            </geometry>
+        </collision>
+    </link>
+    <!-- ________________________________________________________________________________ -->
+    <link name="phalanx_forefinger_2_link">
+        <xacro:default_inertial mass="0.01"/>
+        <visual>
+            <origin xyz="0.0 0.0 0.0" rpy="0.0 0.0 0.0"/>
+            <geometry>
+                <mesh filename="package://arm_description/mesh/phalanx_finger_2.STL" scale="0.3 0.3 0.3"/>
+            </geometry>
+            <material name="LightGrey">
+                <color rgba="0.7 0.7 0.7 1.0"/>
+            </material>
+        </visual>
+        <collision>
+            <origin xyz="0.0 0.0 0.0" rpy="0.0 0.0 0.0"/>
+            <geometry>
+                <mesh filename="package://arm_description/mesh/phalanx_finger_2.STL" scale="0.3 0.3 0.3"/>
+            </geometry>
+        </collision>
+    </link>
+    <!-- ________________________________________________________________________________ -->
+    <link name="phalanx_forefinger_3_link">
+        <xacro:default_inertial mass="0.01"/>
+        <visual>
+            <origin xyz="0.0 0.0 0.0" rpy="0.0 0.0 0.0"/>
+            <geometry>
+                <mesh filename="package://arm_description/mesh/phalanx_finger_3.STL" scale="0.3 0.3 0.3"/>
+            </geometry>
+            <material name="LightGrey">
+                <color rgba="0.7 0.7 0.7 1.0"/>
+            </material>
+        </visual>
+        <collision>
+            <origin xyz="0.0 0.0 0.0" rpy="0.0 0.0 0.0"/>
+            <geometry>
+                <mesh filename="package://arm_description/mesh/phalanx_finger_3.STL" scale="0.3 0.3 0.3"/>
             </geometry>
         </collision>
@@ -274,4 +654,156 @@
     </joint>
     <!-- ________________________________________________________________________________ -->
+    <joint name="joint_thumb" type="revolute">
+        <parent link="hand_link"/>
+        <child link="thumb_link"/>
+        <origin xyz="0.101 0.009 0.11" rpy="0 0 0"/>
+        <axis xyz="0 0 1"/>
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