Commit message: change material

File: arm_description/urdf/arm.urdf.xacro (robot description, xacro)
@@ -13,4 +13,23 @@
                 <mesh filename="package://arm_description/mesh/stand.STL" scale="0.3 0.3 0.3"/>
             </geometry>
+            <material name="yelloworange" >
+                <color rgba="0.9882352941176471 0.6901960784313725 0.00392156862745098 1.0" />
+            </material>
+        </visual>
+        <collision>
+            <origin xyz="0.0 0.0 0.0" rpy="0.0 0.0 0.0"/>
+            <geometry>
+                <mesh filename="package://arm_description/mesh/stand.STL" scale="0.3 0.3 0.3"/>
+            </geometry>
+        </collision>
+    </link>
+    <!-- ________________________________________________________________________________ -->
+    <link name="shoulder_Y_link">
+        <xacro:default_inertial mass="0.5"/>
+        <visual>
+            <origin xyz="0.0 0.0 -0.001" rpy="0.0 0.0 0.0"/>
+            <geometry>
+                <mesh filename="package://arm_description/mesh/joint_shoulder_Y.STL" scale="0.3 0.3 0.3"/>
+            </geometry>
             <material name="LightGrey">
                 <color rgba="0.7 0.7 0.7 1.0"/>
@@ -18,17 +37,17 @@
         </visual>
         <collision>
-            <origin xyz="0.0 0.0 0.0" rpy="0.0 0.0 0.0"/>
-            <geometry>
-                <mesh filename="package://arm_description/mesh/stand.STL" scale="0.3 0.3 0.3"/>
-            </geometry>
-        </collision>
-    </link>
-    <!-- ________________________________________________________________________________ -->
-    <link name="shoulder_Y_link">
-        <xacro:default_inertial mass="0.5"/>
-        <visual>
             <origin xyz="0.0 0.0 -0.001" rpy="0.0 0.0 0.0"/>
             <geometry>
                 <mesh filename="package://arm_description/mesh/joint_shoulder_Y.STL" scale="0.3 0.3 0.3"/>
+            </geometry>
+        </collision>
+    </link>
+    <!-- ________________________________________________________________________________ -->
+    <link name="shoulder_X_link">
+        <xacro:default_inertial mass="0.2"/>
+        <visual>
+            <origin xyz="0.0 0.0 0.0" rpy="0.0 0.0 0.0"/>
+            <geometry>
+                <mesh filename="package://arm_description/mesh/joint_shoulder_X.STL" scale="0.3 0.3 0.3"/>
             </geometry>
             <material name="LightGrey">
@@ -37,17 +56,36 @@
         </visual>
         <collision>
-            <origin xyz="0.0 0.0 -0.001" rpy="0.0 0.0 0.0"/>
-            <geometry>
-                <mesh filename="package://arm_description/mesh/joint_shoulder_Y.STL" scale="0.3 0.3 0.3"/>
-            </geometry>
-        </collision>
-    </link>
-    <!-- ________________________________________________________________________________ -->
-    <link name="shoulder_X_link">
-        <xacro:default_inertial mass="0.2"/>
-        <visual>
             <origin xyz="0.0 0.0 0.0" rpy="0.0 0.0 0.0"/>
             <geometry>
                 <mesh filename="package://arm_description/mesh/joint_shoulder_X.STL" scale="0.3 0.3 0.3"/>
+            </geometry>
+        </collision>
+    </link>
+    <!-- ________________________________________________________________________________ -->
+    <link name="shoulder_link">
+        <xacro:default_inertial mass="2.0"/>
+        <visual>
+            <origin xyz="0.0 0.0 0.0" rpy="0.0 0.0 0.0"/>
+            <geometry>
+                <mesh filename="package://arm_description/mesh/shoulder.STL" scale="0.3 0.3 0.3"/>
+            </geometry>
+            <material name="blue" >
+                <color rgba="0.011764705882352941 0.2627450980392157 0.8745098039215686 1.0" />
+            </material>
+        </visual>
+        <collision>
+            <origin xyz="0.0 0.0 0.0" rpy="0.0 0.0 0.0"/>
+            <geometry>
+                <mesh filename="package://arm_description/mesh/shoulder.STL" scale="0.3 0.3 0.3"/>
+            </geometry>
+        </collision>
+    </link>
+    <!-- ________________________________________________________________________________ -->
+    <link name="elbow_Z_link">
+        <xacro:default_inertial mass="0.5"/>
+        <visual>
+            <origin xyz="0.0 0.0 0.0" rpy="0.0 0.0 0.0"/>
+            <geometry>
+                <mesh filename="package://arm_description/mesh/joint_elbow_Z.STL" scale="0.3 0.3 0.3"/>
             </geometry>
             <material name="LightGrey">
@@ -58,15 +96,15 @@
             <origin xyz="0.0 0.0 0.0" rpy="0.0 0.0 0.0"/>
             <geometry>
-                <mesh filename="package://arm_description/mesh/joint_shoulder_X.STL" scale="0.3 0.3 0.3"/>
-            </geometry>
-        </collision>
-    </link>
-    <!-- ________________________________________________________________________________ -->
-    <link name="shoulder_link">
-        <xacro:default_inertial mass="2.0"/>
-        <visual>
-            <origin xyz="0.0 0.0 0.0" rpy="0.0 0.0 0.0"/>
-            <geometry>
-                <mesh filename="package://arm_description/mesh/shoulder.STL" scale="0.3 0.3 0.3"/>
+                <mesh filename="package://arm_description/mesh/joint_elbow_Z.STL" scale="0.3 0.3 0.3"/>
+            </geometry>
+        </collision>
+    </link>
+    <!-- ________________________________________________________________________________ -->
+    <link name="elbow_X_link">
+        <xacro:default_inertial mass="0.2"/>
+        <visual>
+            <origin xyz="0.0 0.0 0.0" rpy="0.0 0.0 0.0"/>
+            <geometry>
+                <mesh filename="package://arm_description/mesh/joint_elbow_X.STL" scale="0.3 0.3 0.3"/>
             </geometry>
             <material name="LightGrey">
@@ -77,15 +115,34 @@
             <origin xyz="0.0 0.0 0.0" rpy="0.0 0.0 0.0"/>
             <geometry>
-                <mesh filename="package://arm_description/mesh/shoulder.STL" scale="0.3 0.3 0.3"/>
-            </geometry>
-        </collision>
-    </link>
-    <!-- ________________________________________________________________________________ -->
-    <link name="elbow_Z_link">
-        <xacro:default_inertial mass="0.5"/>
-        <visual>
-            <origin xyz="0.0 0.0 0.0" rpy="0.0 0.0 0.0"/>
-            <geometry>
-                <mesh filename="package://arm_description/mesh/joint_elbow_Z.STL" scale="0.3 0.3 0.3"/>
+                <mesh filename="package://arm_description/mesh/joint_elbow_X.STL" scale="0.3 0.3 0.3"/>
+            </geometry>
+        </collision>
+    </link>
+    <!-- ________________________________________________________________________________ -->
+    <link name="forearm_link">
+        <xacro:default_inertial mass="1.2"/>
+        <visual>
+            <origin xyz="0.0 0.0 0.0" rpy="0.0 0.0 0.0"/>
+            <geometry>
+                <mesh filename="package://arm_description/mesh/forearm.STL" scale="0.3 0.3 0.3"/>
+            </geometry>
+            <material name="blue" >
+                <color rgba="0.011764705882352941 0.2627450980392157 0.8745098039215686 1.0" />
+            </material>
+        </visual>
+        <collision>
+            <origin xyz="0.0 0.0 0.0" rpy="0.0 0.0 0.0"/>
+            <geometry>
+                <mesh filename="package://arm_description/mesh/forearm.STL" scale="0.3 0.3 0.3"/>
+            </geometry>
+        </collision>
+    </link>
+    <!-- ________________________________________________________________________________ -->
+    <link name="wrist_Z_link">
+        <xacro:default_inertial mass="0.2"/>
+        <visual>
+            <origin xyz="0.0 0.0 0.0" rpy="0.0 0.0 0.0"/>
+            <geometry>
+                <mesh filename="package://arm_description/mesh/joint_wrist_Z.STL" scale="0.3 0.3 0.3"/>
             </geometry>
             <material name="LightGrey">
@@ -96,15 +153,15 @@
             <origin xyz="0.0 0.0 0.0" rpy="0.0 0.0 0.0"/>
             <geometry>
-                <mesh filename="package://arm_description/mesh/joint_elbow_Z.STL" scale="0.3 0.3 0.3"/>
-            </geometry>
-        </collision>
-    </link>
-    <!-- ________________________________________________________________________________ -->
-    <link name="elbow_X_link">
+                <mesh filename="package://arm_description/mesh/joint_wrist_Z.STL" scale="0.3 0.3 0.3"/>
+            </geometry>
+        </collision>
+    </link>
+    <!-- ________________________________________________________________________________ -->
+    <link name="wrist_X_link">
         <xacro:default_inertial mass="0.2"/>
         <visual>
             <origin xyz="0.0 0.0 0.0" rpy="0.0 0.0 0.0"/>
             <geometry>
-                <mesh filename="package://arm_description/mesh/joint_elbow_X.STL" scale="0.3 0.3 0.3"/>
+                <mesh filename="package://arm_description/mesh/joint_wrist_X.STL" scale="0.3 0.3 0.3"/>
             </geometry>
             <material name="LightGrey">
@@ -115,61 +172,4 @@
             <origin xyz="0.0 0.0 0.0" rpy="0.0 0.0 0.0"/>
             <geometry>
-                <mesh filename="package://arm_description/mesh/joint_elbow_X.STL" scale="0.3 0.3 0.3"/>
-            </geometry>
-        </collision>
-    </link>
-    <!-- ________________________________________________________________________________ -->
-    <link name="forearm_link">
-        <xacro:default_inertial mass="1.2"/>
-        <visual>
-            <origin xyz="0.0 0.0 0.0" rpy="0.0 0.0 0.0"/>
-            <geometry>
-                <mesh filename="package://arm_description/mesh/forearm.STL" scale="0.3 0.3 0.3"/>
-            </geometry>
-            <material name="LightGrey">
-                <color rgba="0.7 0.7 0.7 1.0"/>
-            </material>
-        </visual>
-        <collision>
-            <origin xyz="0.0 0.0 0.0" rpy="0.0 0.0 0.0"/>
-            <geometry>
-                <mesh filename="package://arm_description/mesh/forearm.STL" scale="0.3 0.3 0.3"/>
-            </geometry>
-        </collision>
-    </link>
-    <!-- ________________________________________________________________________________ -->
-    <link name="wrist_Z_link">
-        <xacro:default_inertial mass="0.2"/>
-        <visual>
-            <origin xyz="0.0 0.0 0.0" rpy="0.0 0.0 0.0"/>
-            <geometry>
-                <mesh filename="package://arm_description/mesh/joint_wrist_Z.STL" scale="0.3 0.3 0.3"/>
-            </geometry>
-            <material name="LightGrey">
-                <color rgba="0.7 0.7 0.7 1.0"/>
-            </material>
-        </visual>
-        <collision>
-            <origin xyz="0.0 0.0 0.0" rpy="0.0 0.0 0.0"/>
-            <geometry>
-                <mesh filename="package://arm_description/mesh/joint_wrist_Z.STL" scale="0.3 0.3 0.3"/>
-            </geometry>
-        </collision>
-    </link>
-    <!-- ________________________________________________________________________________ -->
-    <link name="wrist_X_link">
-        <xacro:default_inertial mass="0.2"/>
-        <visual>
-            <origin xyz="0.0 0.0 0.0" rpy="0.0 0.0 0.0"/>
-            <geometry>
-                <mesh filename="package://arm_description/mesh/joint_wrist_X.STL" scale="0.3 0.3 0.3"/>
-            </geometry>
-            <material name="LightGrey">
-                <color rgba="0.7 0.7 0.7 1.0"/>
-            </material>
-        </visual>
-        <collision>
-            <origin xyz="0.0 0.0 0.0" rpy="0.0 0.0 0.0"/>
-            <geometry>
                 <mesh filename="package://arm_description/mesh/joint_wrist_X.STL" scale="0.3 0.3 0.3"/>
             </geometry>
@@ -184,6 +184,6 @@
                 <mesh filename="package://arm_description/mesh/hand.STL" scale="0.3 0.3 0.3"/>
             </geometry>
-            <material name="LightGrey">
-                <color rgba="0.7 0.7 0.7 1.0"/>
+            <material name="blue" >
+                <color rgba="0.011764705882352941 0.2627450980392157 0.8745098039215686 1.0" />
             </material>
         </visual>
@@ -203,6 +203,6 @@
                 <mesh filename="package://arm_description/mesh/joint_thumb.STL" scale="0.3 0.3 0.3"/>
             </geometry>
-            <material name="LightGrey">
-                <color rgba="0.7 0.7 0.7 1.0"/>
+            <material name="red" >
+                <color rgba="0.8980392156862745 0.0 0.0 1.0" />
             </material>
         </visual>
@@ -222,6 +222,6 @@
                 <mesh filename="package://arm_description/mesh/joint_finger.STL" scale="0.3 0.3 0.3"/>
             </geometry>
-            <material name="LightGrey">
-                <color rgba="0.7 0.7 0.7 1.0"/>
+            <material name="red" >
+                <color rgba="0.8980392156862745 0.0 0.0 1.0" />
             </material>
         </visual>
@@ -241,6 +241,6 @@
                 <mesh filename="package://arm_description/mesh/phalanx_thumb_1.STL" scale="0.3 0.3 0.3"/>
             </geometry>
-            <material name="LightGrey">
-                <color rgba="0.7 0.7 0.7 1.0"/>
+            <material name="red" >
+                <color rgba="0.8980392156862745 0.0 0.0 1.0" />
             </material>
         </visual>
@@ -260,6 +260,6 @@
                 <mesh filename="package://arm_description/mesh/phalanx_thumb_2.STL" scale="0.3 0.3 0.3"/>
             </geometry>
-            <material name="LightGrey">
-                <color rgba="0.7 0.7 0.7 1.0"/>
+            <material name="red" >
+                <color rgba="0.8980392156862745 0.0 0.0 1.0" />
             </material>
         </visual>
@@ -279,6 +279,6 @@
                 <mesh filename="package://arm_description/mesh/joint_finger.STL" scale="0.3 0.3 0.3"/>
             </geometry>
-            <material name="LightGrey">
-                <color rgba="0.7 0.7 0.7 1.0"/>
+            <material name="red" >
+                <color rgba="0.8980392156862745 0.0 0.0 1.0" />
             </material>
         </visual>
@@ -298,6 +298,6 @@
                 <mesh filename="package://arm_description/mesh/phalanx_lit_finger_1.STL" scale="0.3 0.3 0.3"/>
             </geometry>
-            <material name="LightGrey">
-                <color rgba="0.7 0.7 0.7 1.0"/>
+            <material name="red" >
+                <color rgba="0.8980392156862745 0.0 0.0 1.0" />
             </material>
         </visual>
@@ -317,6 +317,6 @@
                 <mesh filename="package://arm_description/mesh/phalanx_lit_finger_2.STL" scale="0.3 0.3 0.3"/>
             </geometry>
-            <material name="LightGrey">
-                <color rgba="0.7 0.7 0.7 1.0"/>
+            <material name="red" >
+                <color rgba="0.8980392156862745 0.0 0.0 1.0" />
             </material>
         </visual>
@@ -336,6 +336,6 @@
                 <mesh filename="package://arm_description/mesh/phalanx_lit_finger_3.STL" scale="0.3 0.3 0.3"/>
             </geometry>
-            <material name="LightGrey">
-                <color rgba="0.7 0.7 0.7 1.0"/>
+            <material name="red" >
+                <color rgba="0.8980392156862745 0.0 0.0 1.0" />
             </material>
         </visual>
@@ -355,6 +355,6 @@
                 <mesh filename="package://arm_description/mesh/joint_finger.STL" scale="0.3 0.3 0.3"/>
             </geometry>
-            <material name="LightGrey">
-                <color rgba="0.7 0.7 0.7 1.0"/>
+            <material name="red" >
+                <color rgba="0.8980392156862745 0.0 0.0 1.0" />
             </material>
         </visual>
@@ -374,6 +374,6 @@
                 <mesh filename="package://arm_description/mesh/phalanx_finger_1.STL" scale="0.3 0.3 0.3"/>
             </geometry>
-            <material name="LightGrey">
-                <color rgba="0.7 0.7 0.7 1.0"/>
+            <material name="red" >
+                <color rgba="0.8980392156862745 0.0 0.0 1.0" />
             </material>
         </visual>
@@ -393,6 +393,6 @@
                 <mesh filename="package://arm_description/mesh/phalanx_finger_2.STL" scale="0.3 0.3 0.3"/>
             </geometry>
-            <material name="LightGrey">
-                <color rgba="0.7 0.7 0.7 1.0"/>
+            <material name="red" >
+                <color rgba="0.8980392156862745 0.0 0.0 1.0" />
             </material>
         </visual>
@@ -412,6 +412,6 @@
                 <mesh filename="package://arm_description/mesh/phalanx_finger_3.STL" scale="0.3 0.3 0.3"/>
             </geometry>
-            <material name="LightGrey">
-                <color rgba="0.7 0.7 0.7 1.0"/>
+            <material name="red" >
+                <color rgba="0.8980392156862745 0.0 0.0 1.0" />
             </material>
         </visual>
@@ -431,6 +431,6 @@
                 <mesh filename="package://arm_description/mesh/joint_finger.STL" scale="0.3 0.3 0.3"/>
             </geometry>
-            <material name="LightGrey">
-                <color rgba="0.7 0.7 0.7 1.0"/>
+            <material name="red" >
+                <color rgba="0.8980392156862745 0.0 0.0 1.0" />
             </material>
         </visual>
@@ -450,6 +450,6 @@
                 <mesh filename="package://arm_description/mesh/phalanx_finger_1.STL" scale="0.3 0.3 0.3"/>
             </geometry>
-            <material name="LightGrey">
-                <color rgba="0.7 0.7 0.7 1.0"/>
+            <material name="red" >
+                <color rgba="0.8980392156862745 0.0 0.0 1.0" />
             </material>
         </visual>
@@ -469,6 +469,6 @@
                 <mesh filename="package://arm_description/mesh/phalanx_finger_2.STL" scale="0.3 0.3 0.3"/>
             </geometry>
-            <material name="LightGrey">
-                <color rgba="0.7 0.7 0.7 1.0"/>
+            <material name="red" >
+                <color rgba="0.8980392156862745 0.0 0.0 1.0" />
             </material>
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