Commit message: add material macro in urdf

File: arm_description/urdf/arm.urdf.xacro (robot description, xacro)
@@ -13,7 +13,5 @@
                 <mesh filename="package://arm_description/mesh/stand.STL" scale="0.3 0.3 0.3"/>
             </geometry>
-            <material name="yelloworange" >
-                <color rgba="0.9882352941176471 0.6901960784313725 0.00392156862745098 1.0" />
-            </material>
+            <xacro:yelloworange_material/>
         </visual>
         <collision>
@@ -32,7 +30,5 @@
                 <mesh filename="package://arm_description/mesh/joint_shoulder_Y.STL" scale="0.3 0.3 0.3"/>
             </geometry>
-            <material name="LightGrey">
-                <color rgba="0.7 0.7 0.7 1.0"/>
-            </material>
+            <xacro:lightgrey_material/>
         </visual>
         <collision>
@@ -51,7 +47,5 @@
                 <mesh filename="package://arm_description/mesh/joint_shoulder_X.STL" scale="0.3 0.3 0.3"/>
             </geometry>
-            <material name="LightGrey">
-                <color rgba="0.7 0.7 0.7 1.0"/>
-            </material>
+            <xacro:lightgrey_material/>
         </visual>
         <collision>
@@ -70,7 +64,5 @@
                 <mesh filename="package://arm_description/mesh/shoulder.STL" scale="0.3 0.3 0.3"/>
             </geometry>
-            <material name="blue" >
-                <color rgba="0.011764705882352941 0.2627450980392157 0.8745098039215686 1.0" />
-            </material>
+            <xacro:blue_material/>
         </visual>
         <collision>
@@ -89,7 +81,5 @@
                 <mesh filename="package://arm_description/mesh/joint_elbow_Z.STL" scale="0.3 0.3 0.3"/>
             </geometry>
-            <material name="LightGrey">
-                <color rgba="0.7 0.7 0.7 1.0"/>
-            </material>
+            <xacro:lightgrey_material/>
         </visual>
         <collision>
@@ -108,7 +98,5 @@
                 <mesh filename="package://arm_description/mesh/joint_elbow_X.STL" scale="0.3 0.3 0.3"/>
             </geometry>
-            <material name="LightGrey">
-                <color rgba="0.7 0.7 0.7 1.0"/>
-            </material>
+            <xacro:lightgrey_material/>
         </visual>
         <collision>
@@ -127,7 +115,5 @@
                 <mesh filename="package://arm_description/mesh/forearm.STL" scale="0.3 0.3 0.3"/>
             </geometry>
-            <material name="blue" >
-                <color rgba="0.011764705882352941 0.2627450980392157 0.8745098039215686 1.0" />
-            </material>
+            <xacro:blue_material/>
         </visual>
         <collision>
@@ -146,7 +132,5 @@
                 <mesh filename="package://arm_description/mesh/joint_wrist_Z.STL" scale="0.3 0.3 0.3"/>
             </geometry>
-            <material name="LightGrey">
-                <color rgba="0.7 0.7 0.7 1.0"/>
-            </material>
+            <xacro:lightgrey_material/>
         </visual>
         <collision>
@@ -165,7 +149,5 @@
                 <mesh filename="package://arm_description/mesh/joint_wrist_X.STL" scale="0.3 0.3 0.3"/>
             </geometry>
-            <material name="LightGrey">
-                <color rgba="0.7 0.7 0.7 1.0"/>
-            </material>
+            <xacro:lightgrey_material/>
         </visual>
         <collision>
@@ -184,7 +166,5 @@
                 <mesh filename="package://arm_description/mesh/hand.STL" scale="0.3 0.3 0.3"/>
             </geometry>
-            <material name="blue" >
-                <color rgba="0.011764705882352941 0.2627450980392157 0.8745098039215686 1.0" />
-            </material>
+            <xacro:blue_material/>
         </visual>
         <collision>
@@ -203,7 +183,5 @@
                 <mesh filename="package://arm_description/mesh/joint_thumb.STL" scale="0.3 0.3 0.3"/>
             </geometry>
-            <material name="red" >
-                <color rgba="0.8980392156862745 0.0 0.0 1.0" />
-            </material>
+            <xacro:red_material/>
         </visual>
         <collision>
@@ -222,7 +200,5 @@
                 <mesh filename="package://arm_description/mesh/joint_finger.STL" scale="0.3 0.3 0.3"/>
             </geometry>
-            <material name="red" >
-                <color rgba="0.8980392156862745 0.0 0.0 1.0" />
-            </material>
+            <xacro:red_material/>
         </visual>
         <collision>
@@ -241,7 +217,5 @@
                 <mesh filename="package://arm_description/mesh/phalanx_thumb_1.STL" scale="0.3 0.3 0.3"/>
             </geometry>
-            <material name="red" >
-                <color rgba="0.8980392156862745 0.0 0.0 1.0" />
-            </material>
+            <xacro:red_material/>
         </visual>
         <collision>
@@ -260,7 +234,5 @@
                 <mesh filename="package://arm_description/mesh/phalanx_thumb_2.STL" scale="0.3 0.3 0.3"/>
             </geometry>
-            <material name="red" >
-                <color rgba="0.8980392156862745 0.0 0.0 1.0" />
-            </material>
+            <xacro:red_material/>
         </visual>
         <collision>
@@ -279,7 +251,5 @@
                 <mesh filename="package://arm_description/mesh/joint_finger.STL" scale="0.3 0.3 0.3"/>
             </geometry>
-            <material name="red" >
-                <color rgba="0.8980392156862745 0.0 0.0 1.0" />
-            </material>
+            <xacro:red_material/>
         </visual>
         <collision>
@@ -298,7 +268,5 @@
                 <mesh filename="package://arm_description/mesh/phalanx_lit_finger_1.STL" scale="0.3 0.3 0.3"/>
             </geometry>
-            <material name="red" >
-                <color rgba="0.8980392156862745 0.0 0.0 1.0" />
-            </material>
+            <xacro:red_material/>
         </visual>
         <collision>
@@ -317,7 +285,5 @@
                 <mesh filename="package://arm_description/mesh/phalanx_lit_finger_2.STL" scale="0.3 0.3 0.3"/>
             </geometry>
-            <material name="red" >
-                <color rgba="0.8980392156862745 0.0 0.0 1.0" />
-            </material>
+            <xacro:red_material/>
         </visual>
         <collision>
@@ -336,7 +302,5 @@
                 <mesh filename="package://arm_description/mesh/phalanx_lit_finger_3.STL" scale="0.3 0.3 0.3"/>
             </geometry>
-            <material name="red" >
-                <color rgba="0.8980392156862745 0.0 0.0 1.0" />
-            </material>
+            <xacro:red_material/>
         </visual>
         <collision>
@@ -355,7 +319,5 @@
                 <mesh filename="package://arm_description/mesh/joint_finger.STL" scale="0.3 0.3 0.3"/>
             </geometry>
-            <material name="red" >
-                <color rgba="0.8980392156862745 0.0 0.0 1.0" />
-            </material>
+            <xacro:red_material/>
         </visual>
         <collision>
@@ -374,7 +336,5 @@
                 <mesh filename="package://arm_description/mesh/phalanx_finger_1.STL" scale="0.3 0.3 0.3"/>
             </geometry>
-            <material name="red" >
-                <color rgba="0.8980392156862745 0.0 0.0 1.0" />
-            </material>
+            <xacro:red_material/>
         </visual>
         <collision>
@@ -393,7 +353,5 @@
                 <mesh filename="package://arm_description/mesh/phalanx_finger_2.STL" scale="0.3 0.3 0.3"/>
             </geometry>
-            <material name="red" >
-                <color rgba="0.8980392156862745 0.0 0.0 1.0" />
-            </material>
+            <xacro:red_material/>
         </visual>
         <collision>
@@ -412,7 +370,5 @@
                 <mesh filename="package://arm_description/mesh/phalanx_finger_3.STL" scale="0.3 0.3 0.3"/>
             </geometry>
-            <material name="red" >
-                <color rgba="0.8980392156862745 0.0 0.0 1.0" />
-            </material>
+            <xacro:red_material/>
         </visual>
         <collision>
@@ -431,7 +387,5 @@
                 <mesh filename="package://arm_description/mesh/joint_finger.STL" scale="0.3 0.3 0.3"/>
             </geometry>
-            <material name="red" >
-                <color rgba="0.8980392156862745 0.0 0.0 1.0" />
-            </material>
+            <xacro:red_material/>
         </visual>
         <collision>
@@ -450,7 +404,5 @@
                 <mesh filename="package://arm_description/mesh/phalanx_finger_1.STL" scale="0.3 0.3 0.3"/>
             </geometry>
-            <material name="red" >
-                <color rgba="0.8980392156862745 0.0 0.0 1.0" />
-            </material>
+            <xacro:red_material/>
         </visual>
         <collision>
@@ -469,7 +421,5 @@
                 <mesh filename="package://arm_description/mesh/phalanx_finger_2.STL" scale="0.3 0.3 0.3"/>
             </geometry>
-            <material name="red" >
-                <color rgba="0.8980392156862745 0.0 0.0 1.0" />
-            </material>
+            <xacro:red_material/>
         </visual>
         <collision>
@@ -488,7 +438,5 @@
                 <mesh filename="package://arm_description/mesh/phalanx_finger_3.STL" scale="0.3 0.3 0.3"/>
             </geometry>
-            <material name="red" >
-                <color rgba="0.8980392156862745 0.0 0.0 1.0" />
-            </material>
+            <xacro:red_material/>
         </visual>
         <collision>
@@ -507,7 +455,5 @@
                 <mesh filename="package://arm_description/mesh/joint_finger.STL" scale="0.3 0.3 0.3"/>
             </geometry>
-            <material name="red" >
-                <color rgba="0.8980392156862745 0.0 0.0 1.0" />
-            </material>
+            <xacro:red_material/>
         </visual>
         <collision>
@@ -526,7 +472,5 @@
                 <mesh filename="package://arm_description/mesh/phalanx_finger_1.STL" scale="0.3 0.3 0.3"/>
             </geometry>
-            <material name="red" >
-                <color rgba="0.8980392156862745 0.0 0.0 1.0" />
-            </material>
+            <xacro:red_material/>
         </visual>
         <collision>
@@ -545,7 +489,5 @@
                 <mesh filename="package://arm_description/mesh/phalanx_finger_2.STL" scale="0.3 0.3 0.3"/>
             </geometry>
-            <material name="red" >
-                <color rgba="0.8980392156862745 0.0 0.0 1.0" />
-            </material>
+            <xacro:red_material/>
         </visual>
         <collision>
@@ -564,7 +506,5 @@
                 <mesh filename="package://arm_description/mesh/phalanx_finger_3.STL" scale="0.3 0.3 0.3"/>
             </geometry>
-            <material name="red" >
-                <color rgba="0.8980392156862745 0.0 0.0 1.0" />
-            </material>
+            <xacro:red_material/>
         </visual>
         <collision>
@@ -667,5 +607,5 @@
         <origin xyz="0.057 -0.0059 -0.014" rpy="0 -0.65 0"/>
         <axis xyz="0 1 0"/>
-        <limit lower="-${PI/2}" upper="${PI/2}" effort="${effort}" velocity="${velocity}"/>
+        <limit lower="-${PI/35}" upper="${PI/35}" effort="${effort}" velocity="${velocity}"/>
     </joint>
     <!-- ________________________________________________________________________________ -->
@@ -686,8 +626,10 @@
     </joint>
     <!-- ________________________________________________________________________________ -->
-    <joint name="joint_lit_finger" type="fixed">
+    <joint name="joint_lit_finger" type="revolute">
         <parent link="hand_link"/>
         <child link="lit_finger_link"/>
         <origin xyz="-0.1075 0.005 -0.004" rpy="0 0 0"/>
+        <axis xyz="0 1 0"/>
+        <limit lower="-${PI/35}" upper="${PI/35}" effort="${effort}" velocity="${velocity}"/>
     </joint>
     <!-- ________________________________________________________________________________ -->
@@ -716,8 +658,10 @@
     </joint>
     <!-- ________________________________________________________________________________ -->
-    <joint name="joint_ring_finger" type="fixed">
+    <joint name="joint_ring_finger" type="revolute">
         <parent link="hand_link"/>
         <child link="ring_finger_link"/>
         <origin xyz="-0.035 0.005 -0.017" rpy="0 0 0"/>
+        <axis xyz="0 1 0"/>
+        <limit lower="-${PI/35}" upper="${PI/35}" effort="${effort}" velocity="${velocity}"/>
     </joint>
     <!-- ________________________________________________________________________________ -->
@@ -746,8 +690,10 @@
     </joint>
     <!-- ________________________________________________________________________________ -->
-    <joint name="joint_mid_finger" type="fixed">
+    <joint name="joint_mid_finger" type="revolute">
         <parent link="hand_link"/>
         <child link="mid_finger_link"/>
         <origin xyz="0.035 0.005 -0.024" rpy="0 0 0"/>
+        <axis xyz="0 1 0"/>
+        <limit lower="-${PI/35}" upper="${PI/35}" effort="${effort}" velocity="${velocity}"/>
     </joint>
     <!-- ________________________________________________________________________________ -->
@@ -776,8 +722,10 @@
     </joint>
     <!-- ________________________________________________________________________________ -->
-    <joint name="joint_forefinger" type="fixed">
+    <joint name="joint_forefinger" type="revolute">
         <parent link="hand_link"/>
         <child link="forefinger_link"/>
         <origin xyz="0.105 0.005 -0.016" rpy="0 0 0"/>
+        <axis xyz="0 1 0"/>
+        <limit lower="-${PI/35}" upper="${PI/35}" effort="${effort}" velocity="${velocity}"/>
     </joint>
     <!-- ________________________________________________________________________________ -->

File: arm_description/urdf/macro.urdf.xacro (robot description, xacro)
@@ -7,4 +7,25 @@
             <inertia ixx="1.0" ixy="0.0" ixz="0.0" iyy="1.0" iyz="0.0" izz="1.0"/>
         </inertial>
+    </xacro:macro>
+    <!-- Materials -->
+    <xacro:macro name="yelloworange_material">
+        <material name="yelloworange" >
+            <color rgba="0.9882352941176471 0.6901960784313725 0.00392156862745098 1.0" />
+        </material>
+    </xacro:macro>
+    <xacro:macro name="lightgrey_material">
+        <material name="LightGrey">
+            <color rgba="0.7 0.7 0.7 1.0"/>
+        </material>
+    </xacro:macro>
+    <xacro:macro name="blue_material">
+        <material name="blue" >
+            <color rgba="0.011764705882352941 0.2627450980392157 0.8745098039215686 1.0" />
+        </material>
+    </xacro:macro>
+    <xacro:macro name="red_material">
+        <material name="red" >
+            <color rgba="0.8980392156862745 0.0 0.0 1.0" />
+        </material>
     </xacro:macro>
     <!-- Transmission -->
