Commit message: optimize_urdf

File: arm_description/urdf/arm.urdf.xacro (robot description, xacro)
@@ -6,513 +6,63 @@
     <!-- ________________________________________________________________________________ -->
     <link name="world_link"/>
-    <link name="holder_link">
-        <xacro:default_inertial mass="5"/>
-        <visual>
-            <origin xyz="0.0 0.0 0.0" rpy="0.0 0.0 0.0"/>
-            <geometry>
-                <mesh filename="package://arm_description/mesh/stand.STL" scale="0.3 0.3 0.3"/>
-            </geometry>
-            <xacro:yelloworange_material/>
-        </visual>
-        <collision>
-            <origin xyz="0.0 0.0 0.0" rpy="0.0 0.0 0.0"/>
-            <geometry>
-                <mesh filename="package://arm_description/mesh/stand.STL" scale="0.3 0.3 0.3"/>
-            </geometry>
-        </collision>
-    </link>
-    <!-- ________________________________________________________________________________ -->
-    <link name="shoulder_Y_link">
-        <xacro:default_inertial mass="0.5"/>
-        <visual>
-            <origin xyz="0.0 0.0 -0.001" rpy="0.0 0.0 0.0"/>
-            <geometry>
-                <mesh filename="package://arm_description/mesh/joint_shoulder_Y.STL" scale="0.3 0.3 0.3"/>
-            </geometry>
-            <xacro:lightgrey_material/>
-        </visual>
-        <collision>
-            <origin xyz="0.0 0.0 -0.001" rpy="0.0 0.0 0.0"/>
-            <geometry>
-                <mesh filename="package://arm_description/mesh/joint_shoulder_Y.STL" scale="0.3 0.3 0.3"/>
-            </geometry>
-        </collision>
-    </link>
-    <!-- ________________________________________________________________________________ -->
-    <link name="shoulder_X_link">
-        <xacro:default_inertial mass="0.2"/>
-        <visual>
-            <origin xyz="0.0 0.0 0.0" rpy="0.0 0.0 0.0"/>
-            <geometry>
-                <mesh filename="package://arm_description/mesh/joint_shoulder_X.STL" scale="0.3 0.3 0.3"/>
-            </geometry>
-            <xacro:lightgrey_material/>
-        </visual>
-        <collision>
-            <origin xyz="0.0 0.0 0.0" rpy="0.0 0.0 0.0"/>
-            <geometry>
-                <mesh filename="package://arm_description/mesh/joint_shoulder_X.STL" scale="0.3 0.3 0.3"/>
-            </geometry>
-        </collision>
-    </link>
-    <!-- ________________________________________________________________________________ -->
-    <link name="shoulder_link">
-        <xacro:default_inertial mass="2.0"/>
-        <visual>
-            <origin xyz="0.0 0.0 0.0" rpy="0.0 0.0 0.0"/>
-            <geometry>
-                <mesh filename="package://arm_description/mesh/shoulder.STL" scale="0.3 0.3 0.3"/>
-            </geometry>
-            <xacro:blue_material/>
-        </visual>
-        <collision>
-            <origin xyz="0.0 0.0 0.0" rpy="0.0 0.0 0.0"/>
-            <geometry>
-                <mesh filename="package://arm_description/mesh/shoulder.STL" scale="0.3 0.3 0.3"/>
-            </geometry>
-        </collision>
-    </link>
-    <!-- ________________________________________________________________________________ -->
-    <link name="elbow_Z_link">
-        <xacro:default_inertial mass="0.5"/>
-        <visual>
-            <origin xyz="0.0 0.0 0.0" rpy="0.0 0.0 0.0"/>
-            <geometry>
-                <mesh filename="package://arm_description/mesh/joint_elbow_Z.STL" scale="0.3 0.3 0.3"/>
-            </geometry>
-            <xacro:lightgrey_material/>
-        </visual>
-        <collision>
-            <origin xyz="0.0 0.0 0.0" rpy="0.0 0.0 0.0"/>
-            <geometry>
-                <mesh filename="package://arm_description/mesh/joint_elbow_Z.STL" scale="0.3 0.3 0.3"/>
-            </geometry>
-        </collision>
-    </link>
-    <!-- ________________________________________________________________________________ -->
-    <link name="elbow_X_link">
-        <xacro:default_inertial mass="0.2"/>
-        <visual>
-            <origin xyz="0.0 0.0 0.0" rpy="0.0 0.0 0.0"/>
-            <geometry>
-                <mesh filename="package://arm_description/mesh/joint_elbow_X.STL" scale="0.3 0.3 0.3"/>
-            </geometry>
-            <xacro:lightgrey_material/>
-        </visual>
-        <collision>
-            <origin xyz="0.0 0.0 0.0" rpy="0.0 0.0 0.0"/>
-            <geometry>
-                <mesh filename="package://arm_description/mesh/joint_elbow_X.STL" scale="0.3 0.3 0.3"/>
-            </geometry>
-        </collision>
-    </link>
-    <!-- ________________________________________________________________________________ -->
-    <link name="forearm_link">
-        <xacro:default_inertial mass="1.2"/>
-        <visual>
-            <origin xyz="0.0 0.0 0.0" rpy="0.0 0.0 0.0"/>
-            <geometry>
-                <mesh filename="package://arm_description/mesh/forearm.STL" scale="0.3 0.3 0.3"/>
-            </geometry>
-            <xacro:blue_material/>
-        </visual>
-        <collision>
-            <origin xyz="0.0 0.0 0.0" rpy="0.0 0.0 0.0"/>
-            <geometry>
-                <mesh filename="package://arm_description/mesh/forearm.STL" scale="0.3 0.3 0.3"/>
-            </geometry>
-        </collision>
-    </link>
-    <!-- ________________________________________________________________________________ -->
-    <link name="wrist_Z_link">
-        <xacro:default_inertial mass="0.2"/>
-        <visual>
-            <origin xyz="0.0 0.0 0.0" rpy="0.0 0.0 0.0"/>
-            <geometry>
-                <mesh filename="package://arm_description/mesh/joint_wrist_Z.STL" scale="0.3 0.3 0.3"/>
-            </geometry>
-            <xacro:lightgrey_material/>
-        </visual>
-        <collision>
-            <origin xyz="0.0 0.0 0.0" rpy="0.0 0.0 0.0"/>
-            <geometry>
-                <mesh filename="package://arm_description/mesh/joint_wrist_Z.STL" scale="0.3 0.3 0.3"/>
-            </geometry>
-        </collision>
-    </link>
-    <!-- ________________________________________________________________________________ -->
-    <link name="wrist_X_link">
-        <xacro:default_inertial mass="0.2"/>
-        <visual>
-            <origin xyz="0.0 0.0 0.0" rpy="0.0 0.0 0.0"/>
-            <geometry>
-                <mesh filename="package://arm_description/mesh/joint_wrist_X.STL" scale="0.3 0.3 0.3"/>
-            </geometry>
-            <xacro:lightgrey_material/>
-        </visual>
-        <collision>
-            <origin xyz="0.0 0.0 0.0" rpy="0.0 0.0 0.0"/>
-            <geometry>
-                <mesh filename="package://arm_description/mesh/joint_wrist_X.STL" scale="0.3 0.3 0.3"/>
-            </geometry>
-        </collision>
-    </link>
-    <!-- ________________________________________________________________________________ -->
-    <link name="hand_link">
-        <xacro:default_inertial mass="0.1"/>
-        <visual>
-            <origin xyz="0.0 0.0 0.0" rpy="0.0 0.0 0.0"/>
-            <geometry>
-                <mesh filename="package://arm_description/mesh/hand.STL" scale="0.3 0.3 0.3"/>
-            </geometry>
-            <xacro:blue_material/>
-        </visual>
-        <collision>
-            <origin xyz="0.0 0.0 0.0" rpy="0.0 0.0 0.0"/>
-            <geometry>
-                <mesh filename="package://arm_description/mesh/hand.STL" scale="0.3 0.3 0.3"/>
-            </geometry>
-        </collision>
-    </link>
-    <!-- ________________________________________________________________________________ -->
-    <link name="thumb_link">
-        <xacro:default_inertial mass="0.01"/>
-        <visual>
-            <origin xyz="0.0 0.0 0.0" rpy="0.0 0.0 0.0"/>
-            <geometry>
-                <mesh filename="package://arm_description/mesh/joint_thumb.STL" scale="0.3 0.3 0.3"/>
-            </geometry>
-            <xacro:red_material/>
-        </visual>
-        <collision>
-            <origin xyz="0.0 0.0 0.0" rpy="0.0 0.0 0.0"/>
-            <geometry>
-                <mesh filename="package://arm_description/mesh/joint_thumb.STL" scale="0.3 0.3 0.3"/>
-            </geometry>
-        </collision>
-    </link>
-    <!-- ________________________________________________________________________________ -->
-    <link name="thumb_finger_link">
-        <xacro:default_inertial mass="0.01"/>
-        <visual>
-            <origin xyz="0.0 0.0 0.0" rpy="0.0 0.0 0.0"/>
-            <geometry>
-                <mesh filename="package://arm_description/mesh/joint_finger.STL" scale="0.3 0.3 0.3"/>
-            </geometry>
-            <xacro:red_material/>
-        </visual>
-        <collision>
-            <origin xyz="0.0 0.0 0.0" rpy="0.0 0.0 0.0"/>
-            <geometry>
-                <mesh filename="package://arm_description/mesh/joint_finger_thumb.STL" scale="0.3 0.3 0.3"/>
-            </geometry>
-        </collision>
-    </link>
-    <!-- ________________________________________________________________________________ -->
-    <link name="phalanx_thumb_1_link">
-        <xacro:default_inertial mass="0.01"/>
-        <visual>
-            <origin xyz="0.0 0.0 0.0" rpy="0.0 0.0 0.0"/>
-            <geometry>
-                <mesh filename="package://arm_description/mesh/phalanx_thumb_1.STL" scale="0.3 0.3 0.3"/>
-            </geometry>
-            <xacro:red_material/>
-        </visual>
-        <collision>
-            <origin xyz="0.0 0.0 0.0" rpy="0.0 0.0 0.0"/>
-            <geometry>
-                <mesh filename="package://arm_description/mesh/phalanx_thumb_1.STL" scale="0.3 0.3 0.3"/>
-            </geometry>
-        </collision>
-    </link>
-    <!-- ________________________________________________________________________________ -->
-    <link name="phalanx_thumb_2_link">
-        <xacro:default_inertial mass="0.01"/>
-        <visual>
-            <origin xyz="0.0 0.0 0.0" rpy="0.0 0.0 0.0"/>
-            <geometry>
-                <mesh filename="package://arm_description/mesh/phalanx_thumb_2.STL" scale="0.3 0.3 0.3"/>
-            </geometry>
-            <xacro:red_material/>
-        </visual>
-        <collision>
-            <origin xyz="0.0 0.0 0.0" rpy="0.0 0.0 0.0"/>
-            <geometry>
-                <mesh filename="package://arm_description/mesh/phalanx_thumb_2.STL" scale="0.3 0.3 0.3"/>
-            </geometry>
-        </collision>
-    </link>
-    <!-- ________________________________________________________________________________ -->
-    <link name="lit_finger_link">
-        <xacro:default_inertial mass="0.01"/>
-        <visual>
-            <origin xyz="0.0 0.0 0.0" rpy="0.0 0.0 0.0"/>
-            <geometry>
-                <mesh filename="package://arm_description/mesh/joint_finger.STL" scale="0.3 0.3 0.3"/>
-            </geometry>
-            <xacro:red_material/>
-        </visual>
-        <collision>
-            <origin xyz="0.0 0.0 0.0" rpy="0.0 0.0 0.0"/>
-            <geometry>
-                <mesh filename="package://arm_description/mesh/joint_finger.STL" scale="0.3 0.3 0.3"/>
-            </geometry>
-        </collision>
-    </link>
-    <!-- ________________________________________________________________________________ -->
-    <link name="phalanx_lit_finger_1_link">
-        <xacro:default_inertial mass="0.01"/>
-        <visual>
-            <origin xyz="0.0 0.0 0.0" rpy="0.0 0.0 0.0"/>
-            <geometry>
-                <mesh filename="package://arm_description/mesh/phalanx_lit_finger_1.STL" scale="0.3 0.3 0.3"/>
-            </geometry>
-            <xacro:red_material/>
-        </visual>
-        <collision>
-            <origin xyz="0.0 0.0 0.0" rpy="0.0 0.0 0.0"/>
-            <geometry>
-                <mesh filename="package://arm_description/mesh/phalanx_lit_finger_1.STL" scale="0.3 0.3 0.3"/>
-            </geometry>
-        </collision>
-    </link>
-    <!-- ________________________________________________________________________________ -->
-    <link name="phalanx_lit_finger_2_link">
-        <xacro:default_inertial mass="0.01"/>
-        <visual>
-            <origin xyz="0.0 0.0 0.0" rpy="0.0 0.0 0.0"/>
-            <geometry>
-                <mesh filename="package://arm_description/mesh/phalanx_lit_finger_2.STL" scale="0.3 0.3 0.3"/>
-            </geometry>
-            <xacro:red_material/>
-        </visual>
-        <collision>
-            <origin xyz="0.0 0.0 0.0" rpy="0.0 0.0 0.0"/>
-            <geometry>
-                <mesh filename="package://arm_description/mesh/phalanx_lit_finger_2.STL" scale="0.3 0.3 0.3"/>
-            </geometry>
-        </collision>
-    </link>
-    <!-- ________________________________________________________________________________ -->
-    <link name="phalanx_lit_finger_3_link">
-        <xacro:default_inertial mass="0.01"/>
-        <visual>
-            <origin xyz="0.0 0.0 0.0" rpy="0.0 0.0 0.0"/>
-            <geometry>
-                <mesh filename="package://arm_description/mesh/phalanx_lit_finger_3.STL" scale="0.3 0.3 0.3"/>
-            </geometry>
-            <xacro:red_material/>
-        </visual>
-        <collision>
-            <origin xyz="0.0 0.0 0.0" rpy="0.0 0.0 0.0"/>
-            <geometry>
-                <mesh filename="package://arm_description/mesh/phalanx_lit_finger_3.STL" scale="0.3 0.3 0.3"/>
-            </geometry>
-        </collision>
-    </link>
-    <!-- ________________________________________________________________________________ -->
-    <link name="ring_finger_link">
-        <xacro:default_inertial mass="0.01"/>
-        <visual>
-            <origin xyz="0.0 0.0 0.0" rpy="0.0 0.0 0.0"/>
-            <geometry>
-                <mesh filename="package://arm_description/mesh/joint_finger.STL" scale="0.3 0.3 0.3"/>
-            </geometry>
-            <xacro:red_material/>
-        </visual>
-        <collision>
-            <origin xyz="0.0 0.0 0.0" rpy="0.0 0.0 0.0"/>
-            <geometry>
-                <mesh filename="package://arm_description/mesh/joint_finger.STL" scale="0.3 0.3 0.3"/>
-            </geometry>
-        </collision>
-    </link>
-    <!-- ________________________________________________________________________________ -->
-    <link name="phalanx_ring_finger_1_link">
-        <xacro:default_inertial mass="0.01"/>
-        <visual>
-            <origin xyz="0.0 0.0 0.0" rpy="0.0 0.0 0.0"/>
-            <geometry>
-                <mesh filename="package://arm_description/mesh/phalanx_finger_1.STL" scale="0.3 0.3 0.3"/>
-            </geometry>
-            <xacro:red_material/>
-        </visual>
-        <collision>
-            <origin xyz="0.0 0.0 0.0" rpy="0.0 0.0 0.0"/>
-            <geometry>
-                <mesh filename="package://arm_description/mesh/phalanx_finger_1.STL" scale="0.3 0.3 0.3"/>
-            </geometry>
-        </collision>
-    </link>
-    <!-- ________________________________________________________________________________ -->
-    <link name="phalanx_ring_finger_2_link">
-        <xacro:default_inertial mass="0.01"/>
-        <visual>
-            <origin xyz="0.0 0.0 0.0" rpy="0.0 0.0 0.0"/>
-            <geometry>
-                <mesh filename="package://arm_description/mesh/phalanx_finger_2.STL" scale="0.3 0.3 0.3"/>
-            </geometry>
-            <xacro:red_material/>
-        </visual>
-        <collision>
-            <origin xyz="0.0 0.0 0.0" rpy="0.0 0.0 0.0"/>
-            <geometry>
-                <mesh filename="package://arm_description/mesh/phalanx_finger_2.STL" scale="0.3 0.3 0.3"/>
-            </geometry>
-        </collision>
-    </link>
-    <!-- ________________________________________________________________________________ -->
-    <link name="phalanx_ring_finger_3_link">
-        <xacro:default_inertial mass="0.01"/>
-        <visual>
-            <origin xyz="0.0 0.0 0.0" rpy="0.0 0.0 0.0"/>
-            <geometry>
-                <mesh filename="package://arm_description/mesh/phalanx_finger_3.STL" scale="0.3 0.3 0.3"/>
-            </geometry>
-            <xacro:red_material/>
-        </visual>
-        <collision>
-            <origin xyz="0.0 0.0 0.0" rpy="0.0 0.0 0.0"/>
-            <geometry>
-                <mesh filename="package://arm_description/mesh/phalanx_finger_3.STL" scale="0.3 0.3 0.3"/>
-            </geometry>
-        </collision>
-    </link>
-    <!-- ________________________________________________________________________________ -->
-    <link name="mid_finger_link">
-        <xacro:default_inertial mass="0.01"/>
-        <visual>
-            <origin xyz="0.0 0.0 0.0" rpy="0.0 0.0 0.0"/>
-            <geometry>
-                <mesh filename="package://arm_description/mesh/joint_finger.STL" scale="0.3 0.3 0.3"/>
-            </geometry>
-            <xacro:red_material/>
-        </visual>
-        <collision>
-            <origin xyz="0.0 0.0 0.0" rpy="0.0 0.0 0.0"/>
-            <geometry>
-                <mesh filename="package://arm_description/mesh/joint_finger.STL" scale="0.3 0.3 0.3"/>
-            </geometry>
-        </collision>
-    </link>
-    <!-- ________________________________________________________________________________ -->
-    <link name="phalanx_mid_finger_1_link">
-        <xacro:default_inertial mass="0.01"/>
-        <visual>
-            <origin xyz="0.0 0.0 0.0" rpy="0.0 0.0 0.0"/>
-            <geometry>
-                <mesh filename="package://arm_description/mesh/phalanx_finger_1.STL" scale="0.3 0.3 0.3"/>
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
File: arm_description/urdf/macro.urdf.xacro (robot description, xacro)
@@ -1,31 +1,44 @@
 <?xml version="1.0"?>
 <robot xmlns:xacro="http://www.ros.org/wiki/xacro" name="arm">
-    <!-- Inertial -->
-    <xacro:macro name="default_inertial" params="mass">
-        <inertial>
-            <mass value="${mass}"/>
-            <inertia ixx="1.0" ixy="0.0" ixz="0.0" iyy="1.0" iyz="0.0" izz="1.0"/>
-        </inertial>
-    </xacro:macro>
-    <!-- Materials -->
-    <xacro:macro name="yelloworange_material">
-        <material name="yelloworange" >
-            <color rgba="0.9882352941176471 0.6901960784313725 0.00392156862745098 1.0" />
-        </material>
-    </xacro:macro>
-    <xacro:macro name="lightgrey_material">
-        <material name="LightGrey">
-            <color rgba="0.7 0.7 0.7 1.0"/>
-        </material>
-    </xacro:macro>
-    <xacro:macro name="blue_material">
-        <material name="blue" >
-            <color rgba="0.011764705882352941 0.2627450980392157 0.8745098039215686 1.0" />
-        </material>
-    </xacro:macro>
-    <xacro:macro name="red_material">
-        <material name="red" >
-            <color rgba="0.8980392156862745 0.0 0.0 1.0" />
-        </material>
+    <!-- Links -->
+    <xacro:macro name="link" params="name mass mesh_path mesh_material">
+        <link name="${name}">
+            <inertial>
+                <mass value="${mass}"/>
+                <inertia ixx="1.0" ixy="0.0" ixz="0.0" iyy="1.0" iyz="0.0" izz="1.0"/>
+            </inertial>
+            <visual>
+                <origin xyz="0.0 0.0 0.0" rpy="0.0 0.0 0.0"/>
+                <geometry>
+                    <mesh filename="${mesh_path}" scale="0.3 0.3 0.3"/>
+                </geometry>
+                <xacro:if value="${mesh_material == 'yelloworange'}">
+                    <material name="yelloworange" >
+                        <color rgba="0.9882352941176471 0.6901960784313725 0.00392156862745098 1.0" />
+                    </material>
+                </xacro:if>
+                <xacro:if value="${mesh_material == 'lightgrey'}">
+                    <material name="lightgrey" >
+                        <color rgba="0.7 0.7 0.7 1.0" />
+                    </material>
+                </xacro:if>
+                <xacro:if value="${mesh_material == 'blue'}">
+                    <material name="blue" >
+                        <color rgba="0.011764705882352941 0.2627450980392157 0.8745098039215686 1.0" />
+                    </material>
+                </xacro:if>
+                <xacro:if value="${mesh_material == 'red'}">
+                    <material name="red" >
+                        <color rgba="0.8980392156862745 0.0 0.0 1.0" />
+                    </material>
+                </xacro:if>
+            </visual>
+            <collision>
+                <origin xyz="0.0 0.0 0.0" rpy="0.0 0.0 0.0"/>
+                <geometry>
+                    <mesh filename="${mesh_path}" scale="0.3 0.3 0.3"/>
+                </geometry>
+            </collision>
+        </link>
     </xacro:macro>
     <!-- Transmission -->
