Commit message: add config joint_state and trajectory

File: arm_description/urdf/arm.urdf.xacro (robot description, xacro)
@@ -305,3 +305,36 @@
     <!-- ________________________________________________________________________________ -->
     <!-- Joint end -->
+    <xacro:default_transmission name="joint_shoulder_Y"/>
+    <xacro:default_transmission name="joint_shoulder_X"/>
+    <xacro:default_transmission name="joint_elbow_Z"/>
+    <xacro:default_transmission name="joint_elbow_X"/>
+    <xacro:default_transmission name="joint_wrist_Z"/>
+    <xacro:default_transmission name="joint_wrist_X"/>
+    <xacro:default_transmission name="joint_thumb"/>
+    <xacro:default_transmission name="joint_finger_thumb"/>
+    <xacro:default_transmission name="joint_phalanx_thumb_1"/>
+    <xacro:default_transmission name="joint_phalanx_thumb_2"/>
+    <xacro:default_transmission name="joint_lit_finger"/>
+    <xacro:default_transmission name="joint_phalanx_lit_finger_1"/>
+    <xacro:default_transmission name="joint_phalanx_lit_finger_2"/>
+    <xacro:default_transmission name="joint_phalanx_lit_finger_3"/>
+    <xacro:default_transmission name="joint_ring_finger"/>
+    <xacro:default_transmission name="joint_phalanx_ring_finger_1"/>
+    <xacro:default_transmission name="joint_phalanx_ring_finger_2"/>
+    <xacro:default_transmission name="joint_phalanx_ring_finger_3"/>
+    <xacro:default_transmission name="joint_mid_finger"/>
+    <xacro:default_transmission name="joint_phalanx_mid_finger_1"/>
+    <xacro:default_transmission name="joint_phalanx_mid_finger_2"/>
+    <xacro:default_transmission name="joint_phalanx_mid_finger_3"/>
+    <xacro:default_transmission name="joint_forefinger"/>
+    <xacro:default_transmission name="joint_phalanx_forefinger_1"/>
+    <xacro:default_transmission name="joint_phalanx_forefinger_2"/>
+    <xacro:default_transmission name="joint_phalanx_forefinger_3"/>
+    <gazebo>
+        <plugin name="gazebo_ros_control" filename="libgazebo_ros_control.so">
+            <robotNamespace>/arm</robotNamespace>
+            <robotSimType>gazebo_ros_control/DefaultRobotHWSim</robotSimType>
+            <legacyModeNS>true</legacyModeNS>
+        </plugin>
+    </gazebo>
 </robot>

File: arm_description/urdf/macro.urdf.xacro (robot description, xacro)
@@ -43,13 +43,13 @@
     </xacro:macro>
     <!-- Transmission -->
-    <xacro:macro name="default_transmission" params="number">
-        <transmission name="transmission_${number}">
+    <xacro:macro name="default_transmission" params="name">
+        <transmission name="transmission_${name}">
             <type>
                 transmission_interface/SimpleTransmission
             </type>
-            <joint name="joint_${number}">
+            <joint name="${name}">
                 <hardwareInterface>hardware_interface/PositionJointInterface</hardwareInterface>
             </joint>
-            <actuator name="motor_${number}">
+            <actuator name="motor_${name}">
                 <hardwareInterface>hardware_interface/PositionJointInterface</hardwareInterface>
                 <mechanicalReduction>1</mechanicalReduction>

Commit message: add macro for material

File: arm_description/urdf/arm.urdf.xacro (robot description, xacro)
@@ -6,4 +6,17 @@
     <!-- ________________________________________________________________________________ -->
     <link name="world_link"/>
+    <link name="base_link">
+        <visual>
+            <geometry>
+                <cylinder radius="0.5" length="0.1"/>
+            </geometry>
+            <xacro:yelloworange_material/>
+        </visual>
+        <collision>
+            <geometry>
+                <cylinder radius="0.5" length="0.1"/>
+            </geometry>
+        </collision>
+    </link>
     <xacro:link name="holder_link" mass="5" mesh_path="package://arm_description/mesh/stand.STL" mesh_material="yelloworange"/>
     <!-- ________________________________________________________________________________ -->
@@ -71,4 +84,10 @@
     <joint name="virtual_joint" type="fixed">
         <parent link="world_link"/>
+        <child link="base_link"/>
+        <origin xyz="0 0 0.1" rpy="0 0 0"/>
+    </joint>
+<!-- ________________________________________________________________________________ -->
+    <joint name="base_joint" type="fixed">
+        <parent link="base_link"/>
         <child link="holder_link"/>
         <origin xyz="0 0 0" rpy="0 0 0"/>

File: arm_description/urdf/macro.urdf.xacro (robot description, xacro)
@@ -1,4 +1,25 @@
 <?xml version="1.0"?>
 <robot xmlns:xacro="http://www.ros.org/wiki/xacro" name="arm">
+    <!-- Materials -->
+    <xacro:macro name="yelloworange_material">
+        <material name="yelloworange" >
+            <color rgba="0.9882352941176471 0.6901960784313725 0.00392156862745098 1.0" />
+        </material>
+    </xacro:macro>
+    <xacro:macro name="lightgrey_material">
+        <material name="lightgrey" >
+            <color rgba="0.7 0.7 0.7 1.0" />
+        </material>
+    </xacro:macro>
+    <xacro:macro name="blue_material">
+        <material name="blue" >
+            <color rgba="0.011764705882352941 0.2627450980392157 0.8745098039215686 1.0" />
+        </material>
+    </xacro:macro>
+    <xacro:macro name="red_material">
+        <material name="red" >
+            <color rgba="0.8980392156862745 0.0 0.0 1.0" />
+        </material>
+    </xacro:macro>
     <!-- Links -->
     <xacro:macro name="link" params="name mass mesh_path mesh_material">
@@ -14,22 +35,14 @@
                 </geometry>
                 <xacro:if value="${mesh_material == 'yelloworange'}">
-                    <material name="yelloworange" >
-                        <color rgba="0.9882352941176471 0.6901960784313725 0.00392156862745098 1.0" />
-                    </material>
+                    <xacro:yelloworange_material/>
                 </xacro:if>
                 <xacro:if value="${mesh_material == 'lightgrey'}">
-                    <material name="lightgrey" >
-                        <color rgba="0.7 0.7 0.7 1.0" />
-                    </material>
+                    <xacro:lightgrey_material/>
                 </xacro:if>
                 <xacro:if value="${mesh_material == 'blue'}">
-                    <material name="blue" >
-                        <color rgba="0.011764705882352941 0.2627450980392157 0.8745098039215686 1.0" />
-                    </material>
+                    <xacro:blue_material/>
                 </xacro:if>
                 <xacro:if value="${mesh_material == 'red'}">
-                    <material name="red" >
-                        <color rgba="0.8980392156862745 0.0 0.0 1.0" />
-                    </material>
+                    <xacro:red_material/>
                 </xacro:if>
             </visual>
